Commit message: Fix robot xacro and hw's CAN ID
The dirtction of knee_joint  is fixed.
And, CAN IDs used in RobotHW are fixed.

File: leg_robot_moveit/xacro/leg_robot.xacro (robot description, xacro)
@@ -151,5 +151,5 @@
         <axis xyz="0 0 1"/>
         <limit lower="${radians(-150)}" upper="${radians(150)}" velocity="50.0" effort="1000.0"/>
-        <origin xyz="0.3 0 0" rpy="${radians(180)} 0 0"/>
+        <origin xyz="0.3 0 0" rpy="0 0 0"/>
         <dynamics damping="1.0"/>
     </joint>
@@ -170,5 +170,5 @@
         </inertial>
         <visual>
-            <origin xyz="0.0 0.0 0.0" rpy="0.0 0.0 0.0"/>
+            <origin xyz="0.0 0.0 0.0" rpy="${radians(180)} 0.0 0.0"/>
             <geometry>
                 <mesh filename="package://lily_dog/stl/leg_tester/lower_leg_link.stl"/>
